File: vcfvca/vcfvca.sch (EAGLE design)
At the start: 3 parts

Commit message: Draw schematics for the filter and VCA, excluding control
Parts:
- added C10, C11, C7: 6u8, rcl:CPOL-EUE1.8-4
- added C3, C4, C5, C6: 300p MICA, rcl:C-EU050-025X075
- added C8: 100n, rcl:C-EU050-025X075
- added C9: 300p, rcl:C-EU050-025X075
- added IC1, IC3, IC4: LM13700N, national-semiconductor:LM13600N
- added IC2: LM4558N, linear:LM4558N
- added Q1, Q2, Q4, Q5: BF245, transistor-small-signal:BF245
- added Q3, Q6: 2N3906, transistor-small-signal:2N3906
- added R1, R11, R17, R23, R7: 10k, rcl:R-US_0207/10
- added R10, R15, R16, R21, R22, R27, R4, R9: 220R, rcl:R-US_0207/10
- added R12, R18, R20, R24, R33, R5, R8: 100k, rcl:R-US_0207/10
- added R13, R14, R19, R25, R36, R6: 15k, rcl:R-US_0207/10
- added R2: 470k, rcl:R-US_0207/10
- added R26: 33k, rcl:R-US_0207/10
- added R28: 12k, rcl:R-US_0207/10
- added R29, R38: 1k, rcl:R-US_0207/10
- added R3: 100R, rcl:R-US_0207/10
- added R30: 4k7, rcl:R-US_0207/10
- added R31, R32, R35: 1M, rcl:R-US_0207/10
- added R34: 510R, rcl:R-US_0207/10
- added R37: 22k, rcl:R-US_0207/10
- added S1: 12dB/24dB, switch:TL36PO
- added VR1, VR2: 100k, pot:TRIM_US-S63P
Connections:
- new net I_AMP: R36.2
- new net I_FREQ: R11.2, R17.1, R23.1, R7.2
- new net I_RES: R29.2
- new net N$10: IC1B.AMP/BIAS, R11.1
- new net N$11: IC1B.+IN, R9.1
- new net N$12: IC1B.-IN, R10.1, R12.1, R8.2
- new net N$13: C7.+, R30.1
- new net N$14: IC3A.+IN, R14.2, R15.1
- new net N$15: IC3A.-IN, R16.1, R18.1
- new net N$16: IC4A.-IN, R26.2, R27.1
- new net N$17: Q4.S, R18.2, R19.1, R20.1
- new net N$18: Q2.S, Q3.C, R12.2, R13.1, R14.1, S1.S
- new net N$19: Q5.S, Q6.C, R24.2, R25.1, R26.1, S1.O
- new net N$2: C4.1, IC1B.OUT, Q2.G
- new net N$20: IC3B.-IN, R20.2, R22.1, R24.1
- new net N$21: IC3B.+IN, R21.1
- new net N$22: IC4A.AMP/BIAS, R29.1
- new net N$23: IC3A.AMP/BIAS, R17.2
- new net N$24: IC3B.AMP/BIAS, R23.2
- new net N$25: IC4A.OUT, R28.1, R30.2
- new net N$26: Q5.D, Q6.B, R32.2
- new net N$27: Q2.D, Q3.B, R31.2
- new net N$28: C8.1, S1.P
- new net N$29: C8.2, R33.1
- new net N$3: C3.1, IC1A.OUT, Q1.G
- new net N$30: IC4B.+IN, R33.2, R34.1, R35.2
- new net N$31: C9.1, IC2A.-IN, IC4B.OUT, R37.1
- new net N$32: R35.1, VR2.S
- new net N$33: IC4B.AMP/BIAS, R36.1
- new net N$34: R2.1, VR1.S
- new net N$35: C9.2, IC2A.OUT, R37.2, R38.1
- new net N$36: C10.+, R38.2
- new net N$37: C11.+, R1.2
- new net N$4: C5.1, IC3A.OUT, Q4.G
- new net N$5: C6.1, IC3B.OUT, Q5.G
- new net N$6: IC1A.-IN, R2.2, R4.1, R5.1
- new net N$7: IC1A.AMP/BIAS, R7.1
- new net N$8: Q1.S, R5.2, R6.1, R8.1
- new net N$9: C11.-, C7.-, IC1A.+IN, R3.1
- net +15V: now also Q1.D, Q3.E, Q4.D, Q6.E, R31.1, R32.1, VR1.E, VR2.E
- net -15V: now also R13.2, R19.2, R25.2, R6.2, VR1.A, VR2.A
- net GND: now also C3.2, C4.2, C5.2, C6.2, IC2A.+IN, IC4A.+IN, IC4B.-IN, R10.2, R15.2, R16.2, R21.2, R22.2, R27.2, R28.2, R3.2, R34.2, R4.2, R9.2
Other:
- moved on the sheet: C1, C2, J1
